File: uAmp.kicad_sch (KiCad schematic)
At the start: 18 parts, among them J1 PinHeader_1x07, U1 THAT1512P08-U

Commit message: Rename to uAmp; rev3 layout rework, C6 part number, rev2-style render
- Project renamed thatmicpre -> uAmp (files, README title, backups ignore).
- Layout (owner): U1, RV1, C5-C8, R1, R2, R4, R6 moved; GND pour now on
  both layers; header silk relabelled OUT/GND/+15V/-15V/GND/IN-/IN+;
  "uAmp" and "REV.3" added.
- Tidy after the moves: unfillet, collapse drag stubs, redraw seven
  jogged runs (U1 pins 2/3/4/6/7, R4-C7, C6 pad 1) as clean 45-degree
  paths, delete an accidental B.Cu duplicate of the +15V J1-R4 run, J1
  pad 6 solid to the pour, then re-fillet (one corner by RV1 at 0.8 mm
  to keep clearance). Placement, silk and pour untouched by the tidy.
  DRC with schematic parity: 0 errors, 0 unconnected, 0 parity.
- C6 = Nichicon UVZ0J682MHD (6800 uF 6.3 V, 12.5 x 25 mm, 5 mm pitch) in
  schematic, board and BOM; polarized is correct at zero bias, and no
  bipolar 6800 uF fits the footprint.
- README: SSM2019 substitution notes (owner).
- uAmp_rev3_render.png: the rev2 Blender scene (camera, tuned lights,
  world, shadow catcher) with the rev3 board swapped in and per-resistor
  colour bands, composited in Photoshop with the owner's backdrop and
  grade (the PSD is not in the repo). schematic.pdf regenerated.

Co-Authored-By: Claude Opus 5.5 <noreply@anthropic.com>
Parts:
- C6: Vendor (none) -> UVZ0J682MHD
Other:
- moved on the sheet: C3, R1, R2
